File: CMeterFront.kicad_pcb (KiCad board)
At the start: 2 copper layers, 74.4 x 84.7 mm, 48 parts, among them J1 PCB_CONN, J2 PLD-6, Q2 Q_NPN_BCE, Q3 Q_NPN_BCE, Q4 Q_NPN_BCE, SW1 PLUS, SW2 MINUS, T1 L_Measure, U1 ATMEGA8A-PU, U2 BC56-12SRWA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

Commit message: update
Routing:
- net BTN1: track 30.8 -> 29.6 mm
