File: CMeterFront.sch (KiCad schematic (older format))
At the start: 41 parts, among them J1 PCB_CONN, J2 PLD-6, Q2 Q_NPN_BCE, Q3 Q_NPN_BCE, Q4 Q_NPN_BCE, SW1 SW_Push, SW2 SW_Push, U1 ATMEGA8A-PU, U2 BC56-12SRWA, Y1 8Mhz

Commit message: internal milling areas changed for jlcpcb
Parts:
- U1: value ATMEGA8A-PU -> ATMEGA8L
Changed lines of the file:
@@
 P 2600 5750
 F 0 "U1" H 1850 7050 50  0000 L BNN
-F 1 "ATMEGA8A-PU" H 3100 4300 50  0000 L BNN
+F 1 "ATMEGA8L" H 3100 4300 50  0000 L BNN
 F 2 "MyFootprints:TRS-28_Connfly" H 2600 5750 50  0001 C CIN
 F 3 "https://www.chipdip.ru/product/atmega8a-pu" H 2600 5750 50  0001 C CNN
